Commit message: feature: Phase 2a goalie smooth blending + world file ball fix
Phase 2a (goalie idle bias fix):
- ollama_sandbox_bridge.py: read 'role' from strategy JSON, add 10
  field-size-relative GOALIE_* blending parameters (as % of field
  half-length/width), smoothstep() helper at module scope. Goalie
  blending block in state_cb: smooth transition between goal-line
  positioning (ball near) and angle-block (ball far), 70% tactical +
  30% LLM influence, deadband eliminates micro-oscillations.
  Skips when action=='kick' (Part A). Role-aware kick direction:
  goalie clears upfield, non-goalie bots aim at opponent goal (Part B).
  NOTE (Phase 5): blending block removed once Phase 5.1 Kalman
  provides filtered data.
- tools/analyze_trace.py: new goalie_tactical_pct KPI — distinguishes
  'tactically positioning' from 'stuck'. Ball far -> goalie should be
  forward; ball near -> goalie near line + tracking Y.

World file ball fix:
- robocup.world: removed hardcoded soccer_ball model (was always at
  0,0, blocking scenario-specified ball positions). Ball is now spawned
  solely by json_spawner.py from scenario JSON, same as bots.
- football.urdf: ported world-ball physics (mass 0.4, restitution 1.0,
  friction 0.01, velocity_decay 0.002, contact kp/kd/max_vel/min_depth)
  so spawned ball behaves like the old world-file ball.

Scenario:
- scenario/3vs3_goal_kick_blue.json: goal-kick situation for blue
  (ball at -3.5,1.0, goalie at -4.0,1.0, red in own half). Tests goalie
  blending and role-aware kick direction.

Verified: 91 tests pass, 2 headless runs confirmed ball spawns at
scenario position, goalie blends tactically (angle-block forward
when ball far, goal-line when near). Goalie-kick prompt rule deferred
to Phase 4b (game-phase fragment library).

File: core/src/ros2_ws/src/r2k_scenario_spawner/urdf/football.urdf (robot description, URDF)
Before this commit: robot soccer_ball, 1 links, 0 joints
Links:
- link ball_link: mass 0.43 -> 0.4
